File: Frontpanel (LED and stuff)/Frontpanel.sch (KiCad schematic (older format))
At the start: 65 parts

Commit message: Add files via upload
Parts:
- removed C?: 100nF, symbol C
- added C?: 100nF, symbol C
- added J?: CONN_01X08, symbol CONN_01X10
- added J?: Eventuelle LED's, symbol CONN_01X04
- added R? (x5): 120, symbol R
- added R? (x5): 10k, symbol R
- added U? (x2): LTV-827, Housings_DIP:DIP-8_W7.62mm, symbol LTV-827
- added U?: LTV-817, Housings_DIP:DIP-4_W7.62mm, symbol LTV-817
- U? (x4): symbol 74HC595 -> 74HC595-RESCUE-Frontpanel
Connections:
- net DATA_IN: now also J?.9 (P9), R?.2; no longer U?.14 (SER)
- net DATA_IN_CLK: now also J?.8 (P8), R?.2; no longer U?.11 (SRCLK), U?.11 (SRCLK), U?.11 (SRCLK), U?.11 (SRCLK)
- net GND: now also J?.4 (P4), U?.2, U?.2, U?.2, U?.4, U?.4; no longer C?.2, C?.2, C?.2, C?.2, C?.2, C?.2, CSS.2, C_Comp1.2, C_Comp2.2, Cin.2, D?.2 (A), IC?.20 (GND), IC?.20 (GND), Q?.2 (S), Q?.2 (S), Q?.2 (S), Q?.2 (S), R?.1, R?.1, R?.1, R?.1, R?.2, Reg?.~ (VSense), U?.8 (GND), U?.8 (GND), U?.8 (GND), U?.8 (GND)
- net OUT_ACTIVE: now also J?.6 (P6), R?.2; no longer U?.12 (RCLK), U?.12 (RCLK), U?.12 (RCLK), U?.12 (RCLK)
- net SR_CLEAR: now also J?.7 (P7), R?.2; no longer U?.10 (SRCLR), U?.10 (SRCLR), U?.10 (SRCLR), U?.10 (SRCLR)
- net VCC: now also J?.10 (P10); no longer Cin.1, Reg?.~ (VSense)
- net VDD: now also C?.1, U?.4, U?.6, U?.6, U?.8, U?.8
- net at U?.4 (QE): now also J?.1 (P1)
- net at U?.5 (QF): now also J?.2 (P2)
- net at U?.6 (QG): now also J?.3 (P3)
- net at U?.7 (QH): now also J?.4 (P4)
- net ENABLE_Master renamed ENABLE_Panel
- net ENABLE_Panel: now also R?.2, U?.3
- new net: R?.2, U?.10 (SRCLR), U?.10 (SRCLR), U?.10 (SRCLR), U?.10 (SRCLR), U?.7
- new net: R?.2, U?.11 (SRCLK), U?.11 (SRCLK), U?.11 (SRCLK), U?.11 (SRCLK), U?.5
- new net: R?.2, U?.12 (RCLK), U?.12 (RCLK), U?.12 (RCLK), U?.12 (RCLK), U?.5
- new net: R?.2, U?.14 (SER), U?.7
- new net: R?.1, U?.1 (x3)
- new net: R?.1, U?.3 (x2)
- new net ENABLE_MASTER: J?.5 (P5), R?.2
- new net GNDD: C?.2, C?.2, C?.2, C?.2, C?.2, C?.2, C?.2, CSS.2, C_Comp1.2, C_Comp2.2, Cin.2, D?.2 (A), IC?.20 (GND), IC?.20 (GND), J?.2 (P2), Q?.2 (S), Q?.2 (S), Q?.2 (S), Q?.2 (S), R?.1, R?.1, R?.1, R?.1, R?.1, R?.1, R?.1, R?.1, R?.1, R?.2, Reg?.~ (VSense), U?.8 (GND), U?.8 (GND), U?.8 (GND), U?.8 (GND)
- new net VDDA: Cin.1, J?.3 (P3), Reg?.~ (VSense)
Other:
- note added: "Hier verwendet der LTV 826S\n"
- note added: "VDDA = Gleichgerichtete Spannung von Trafo Nr. 2\n\nVCC = Mikrocontroller-Spannung von 3.3 V\n\nGND = Masse von Mikrocontroller\n\nVDD = Frontpanel-Board-Spannung von 5 V\n\nGNDD = Massepotential Trafo Nr. 2 und Forntpanel-Board"
- moved on the sheet: C?, CSS, C_Comp1, C_Comp2, Cin, D?, IC?, JP?, L?, Q?, R?, Reg?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

Commit message: Add files via upload
Parts:
- removed C? (x2): 100nF, symbol C
- removed C?: 22uF, symbol C
- removed CSS: 8,2nF, symbol C
- removed C_Comp1: 1,5nF 50V, symbol C
- removed C_Comp2: 27pF, symbol C
- removed Cin: 4,7uF, symbol C
- removed D?: B340C, symbol DIODE
- removed J?: CONN_01X08, symbol CONN_01X10
- removed J?: Eventuelle LED's, symbol CONN_01X04
- removed JP?: Jumper_NO_Small, symbol Jumper_NO_Small
- removed L?: L-07HCP 6,8µH, symbol INDUCTOR
- removed R?: 10,2k, symbol R
- removed R?: 1,96k, symbol R
- removed R?: 27,4k, symbol R
- removed R? (x5): 120, symbol R
- removed R? (x5): 10k, symbol R
- removed Reg?: TPS54332, symbol TPS54332
- removed U? (x2): LTV-827, Housings_DIP:DIP-8_W7.62mm, symbol LTV-827
- removed U?: LTV-817, Housings_DIP:DIP-4_W7.62mm, symbol LTV-817
- added C? (x3): 100nF, symbol C
- added C?: 1uF, symbol C
- added D? (x5): LED_ALT, symbol LED_ALT
- added J?: HE10-16, symbol HE10-16
- added J?: Conn_01x04, symbol Conn_01x04
- added R?: 91, symbol R
- added R?: 100k, symbol R
- added R? (x2): 10k, symbol R
- added R? (x4): 110, symbol R
- added SW? (x6): SW_DIP_x01, symbol SW_DIP_x01
- added U?: ICM7555, symbol ICM7555
- R? (x24): value 30 -> 27
- U? (x4): symbol 74HC595-RESCUE-Frontpanel -> 74HC595
Connections:
- net GNDD is gone; now on net GND: C?.2, C?.2, C?.2, C?.2, C?.2, IC?.20 (GND), IC?.20 (GND), Q?.2 (S), Q?.2 (S), Q?.2 (S), Q?.2 (S), R?.1, R?.1, R?.1, R?.1, U?.8 (GND), U?.8 (GND), U?.8 (GND), U?.8 (GND)
- net VCC is gone; now on net VDD: U?.16 (VCC)
- net DATA_IN: now also U?.14 (SER), J?.1
- net DATA_IN_CLK: now also U?.11 (SRCLK), U?.11 (SRCLK), U?.11 (SRCLK), U?.11 (SRCLK), J?.3
- net GND: now also C?.2, C?.2, C?.2, C?.2, D?.1 (K), D?.1 (K), D?.1 (K), D?.1 (K), D?.1 (K), J?.4, R?.1, U?.1 (GND)
- net OUT_ACTIVE: now also U?.12 (RCLK), U?.12 (RCLK), U?.12 (RCLK), U?.12 (RCLK), J?.7
- net SR_CLEAR: now also U?.10 (SRCLR), U?.10 (SRCLR), U?.10 (SRCLR), U?.10 (SRCLR), J?.5
- net VDD: now also C?.1, C?.1, J?.2, R?.2, U?.4 (R), U?.8 (VCC)
- net LED_"Set": now reaches U?.4 (QE)
- net LED_"Set": now also R?.2
- net LED_"EN": now reaches U?.5 (QF)
- net LED_"EN": now also R?.2
- net LED_"CV": now reaches U?.6 (QG)
- net LED_"CV": now also R?.2
- net LED_"CC": now reaches U?.7 (QH)
- net LED_"CC": now also R?.2
- new net: J?.1 (Pin_1), J?.10
- new net: J?.12, J?.2 (Pin_2)
- new net: J?.14, J?.3 (Pin_3)
- new net: J?.16, J?.4 (Pin_4)
- new net: C?.1, R?.1, SW?.1
- new net: R?.1, R?.2, SW?.2, U?.2 (TR), U?.6 (THR)
- new net: D?.2 (A), R?.2
- new net: C?.1, U?.5 (CV)
- new net: D?.2 (A), R?.1 (x4)
- new net ON/OFF_Sleepmode: J?.9, R?.1, R?.2, U?.3 (Q)
Other:
- note added: "Anschluss Drehgeber"
- note added: "LED_Matrix_Ansteuerung"
- note added: "Soft On/Off + Power_On_LED\n"
- note removed: "Hier verwendet der LTV 826S\n"
- note removed: "VDDA = Gleichgerichtete Spannung von Trafo Nr. 2\n\nVCC = Mikrocontroller-Spannung von 3.3 V\n\nGND = Masse von Mikrocontroller\n\nVDD = Frontpanel-Board-Spannung von 5 V\n\nGNDD = Massepotential Trafo Nr. 2 und Forntpanel-Board"
- moved on the sheet: C?, IC?, Q?, R?, U?
